File: Kicad/GC - Temp_Sensor.sch (KiCad schematic (older format))
At the start: 3 parts

Commit message: Passives changed from 0805 to 0603
Parts:
- C1: footprint Capacitors_SMD:C_0805 -> Capacitors_SMD:C_0603
- R14, R15: footprint Resistors_SMD:R_0805 -> Resistors_SMD:R_0603
Changed lines of the file:
@@
 F 0 "R15" V 6000 4200 50  0000 C CNN
 F 1 "10k" V 6100 4200 50  0000 C CNN
-F 2 "Resistors_SMD:R_0805" V 5930 4200 30  0001 C CNN
+F 2 "Resistors_SMD:R_0603" V 5930 4200 30  0001 C CNN
 F 3 "" H 6000 4200 30  0000 C CNN
 	1    6000 4200
@@
 F 0 "C1" H 5750 4300 50  0000 L CNN
 F 1 "2.2uF" H 5756 4115 50  0000 L CNN
-F 2 "Capacitors_SMD:C_0805" H 5788 4050 30  0001 C CNN
+F 2 "Capacitors_SMD:C_0603" H 5788 4050 30  0001 C CNN
 F 3 "" H 5750 4200 60  0000 C CNN
 	1    5750 4200
@@
 F 0 "R14" V 6000 3800 50  0000 C CNN
 F 1 "NTC 10k" V 6100 3800 50  0000 C CNN
-F 2 "Resistors_SMD:R_0805" V 5930 3800 30  0001 C CNN
+F 2 "Resistors_SMD:R_0603" V 5930 3800 30  0001 C CNN
 F 3 "" H 6000 3800 30  0000 C CNN
 	1    6000 3800

Commit message: Adjusting capacitor size/value
Parts:
- C1: Tension (none) -> 25V
Changed lines of the file:
@@
 $Descr A4 11693 8268
 encoding utf-8
-Sheet 8 8
+Sheet 7 8
 Title "Gouach Controller"
 Date "2020-02-03"
@@
 F 2 "Capacitors_SMD:C_0603" H 5788 4050 30  0001 C CNN
 F 3 "" H 5750 4200 60  0000 C CNN
+F 4 "25V" H 5750 4200 50  0001 C CNN "Tension"
 	1    5750 4200
 	1    0    0    -1

Commit message: Fixed libraries issues
Parts:
- C1: footprint Capacitors_SMD:C_0603 -> Capacitor_SMD:C_0603_1608Metric; symbol Device:C -> Gouach_Controller-rescue:C-Device
- R14, R15: footprint Resistors_SMD:R_0603 -> Resistor_SMD:R_0603_1608Metric; symbol Device:R -> Gouach_Controller-rescue:R-Device
Changed lines of the file:
@@
 $EndDescr
 $Comp
-L Device:R R15
+L Gouach_Controller-rescue:R-Device R15
 U 1 1 5426DAA6
 P 6000 4200
 F 0 "R15" V 6000 4200 50  0000 C CNN
 F 1 "10k" V 6100 4200 50  0000 C CNN
-F 2 "Resistors_SMD:R_0603" V 5930 4200 30  0001 C CNN
+F 2 "Resistor_SMD:R_0603_1608Metric" V 5930 4200 30  0001 C CNN
 F 3 "" H 6000 4200 30  0000 C CNN
 	1    6000 4200
@@
 $EndComp
 $Comp
-L Device:C C1
+L Gouach_Controller-rescue:C-Device C1
 U 1 1 5426DADD
 P 5750 4200
@@
 F 0 "C1" H 5750 4300 50  0000 L CNN
 F 1 "2.2uF" H 5756 4115 50  0000 L CNN
-F 2 "Capacitors_SMD:C_0603" H 5788 4050 30  0001 C CNN
+F 2 "Capacitor_SMD:C_0603_1608Metric" H 5788 4050 30  0001 C CNN
 F 3 "" H 5750 4200 60  0000 C CNN
 F 4 "25V" H 5750 4200 50  0001 C CNN "Tension"
@@
 $EndComp
 $Comp
-L power:GND #PWR0102
+L Gouach_Controller-rescue:GND-power #PWR0102
 U 1 1 5426DB25
 P 6000 4450
@@
 	6000 3600 6000 3650
 $Comp
-L power:+3V3 #PWR0127
+L Gouach_Controller-rescue:+3V3-power #PWR0127
 U 1 1 5F1769E4
 P 6000 3600
@@
 $EndComp
 $Comp
-L Device:R R14
+L Gouach_Controller-rescue:R-Device R14
 U 1 1 5426DA2F
 P 6000 3800
 F 0 "R14" V 6000 3800 50  0000 C CNN
 F 1 "NTC 10k" V 6100 3800 50  0000 C CNN
-F 2 "Resistors_SMD:R_0603" V 5930 3800 30  0001 C CNN
+F 2 "Resistor_SMD:R_0603_1608Metric" V 5930 3800 30  0001 C CNN
 F 3 "" H 6000 3800 30  0000 C CNN
 	1    6000 3800
