File: Kicad/GC - CAN.sch (KiCad schematic (older format))
At the start: 3 parts, among them U4 SN65HVD232

Commit message: Passives changed from 0805 to 0603
Parts:
- C4: footprint Capacitors_SMD:C_0805 -> Capacitors_SMD:C_0603
- R16: footprint Resistors_SMD:R_0805 -> Resistors_SMD:R_0603
Changed lines of the file:
@@
 F 0 "R16" V 5100 4100 50  0000 C CNN
 F 1 "120R" V 5200 4100 50  0000 C CNN
-F 2 "Resistors_SMD:R_0805" V 5130 4100 30  0001 C CNN
+F 2 "Resistors_SMD:R_0603" V 5130 4100 30  0001 C CNN
 F 3 "" H 5200 4100 30  0000 C CNN
 	1    5200 4100
@@
 F 0 "C4" H 7200 4200 50  0000 L CNN
 F 1 "100nF" H 7206 4015 50  0000 L CNN
-F 2 "Capacitors_SMD:C_0805" H 7238 3950 30  0001 C CNN
+F 2 "Capacitors_SMD:C_0603" H 7238 3950 30  0001 C CNN
 F 3 "" H 7200 4100 60  0000 C CNN
 	1    7200 4100

Commit message: Adjusting capacitor size/value
Parts:
- C4: Tension (none) -> 50V
Changed lines of the file:
@@
 F 2 "Capacitors_SMD:C_0603" H 7238 3950 30  0001 C CNN
 F 3 "" H 7200 4100 60  0000 C CNN
+F 4 "50V" H 7200 4100 50  0001 C CNN "Tension"
 	1    7200 4100
 	1    0    0    -1

Commit message: Fixed libraries issues
Parts:
- C4: footprint Capacitors_SMD:C_0603 -> Capacitor_SMD:C_0603_1608Metric; symbol Device:C -> Gouach_Controller-rescue:C-Device
- R16: footprint Resistors_SMD:R_0603 -> Resistor_SMD:R_0603_1608Metric; symbol Device:R -> Gouach_Controller-rescue:R-Device
- U4: footprint Housings_SOIC:SOIC-8_3.9x4.9mm_Pitch1.27mm -> Package_SO:SOIC-8_3.9x4.9mm_P1.27mm; symbol Interface_CAN_LIN:SN65HVD232 -> Gouach_Controller-rescue:SN65HVD232-Interface_CAN_LIN
Changed lines of the file:
@@
 $EndDescr
 $Comp
-L Interface_CAN_LIN:SN65HVD232 U4
+L Gouach_Controller-rescue:SN65HVD232-Interface_CAN_LIN U4
 U 1 1 53F59F90
 P 5850 4050
@@
 F 0 "U4" H 6100 4300 50  0000 C CNN
 F 1 "SN65HVD232" H 5900 3700 50  0000 C CNN
-F 2 "Housings_SOIC:SOIC-8_3.9x4.9mm_Pitch1.27mm" H 5850 4050 35  0001 C CIN
+F 2 "Package_SO:SOIC-8_3.9x4.9mm_P1.27mm" H 5850 4050 35  0001 C CIN
 F 3 "SN65HVD232" H 5850 4050 60  0001 C CNN
 F 4 "SN65HVD232" H 5850 4050 50  0001 C CNN "mfg#"
@@
 CAN_TX
 $Comp
-L Device:R R16
+L Gouach_Controller-rescue:R-Device R16
 U 1 1 540030A8
 P 5200 4100
 F 0 "R16" V 5100 4100 50  0000 C CNN
 F 1 "120R" V 5200 4100 50  0000 C CNN
-F 2 "Resistors_SMD:R_0603" V 5130 4100 30  0001 C CNN
+F 2 "Resistor_SMD:R_0603_1608Metric" V 5130 4100 30  0001 C CNN
 F 3 "" H 5200 4100 30  0000 C CNN
 	1    5200 4100
@@
 	5200 4250 5350 4250
 $Comp
-L power:+3V3 #PWR0128
+L Gouach_Controller-rescue:+3V3-power #PWR0128
 U 1 1 5F16972D
 P 7200 3950
@@
 $EndComp
 $Comp
-L power:+3V3 #PWR0129
+L Gouach_Controller-rescue:+3V3-power #PWR0129
 U 1 1 5F169DDB
 P 5850 3750
@@
 $EndComp
 $Comp
-L power:GND #PWR0130
+L Gouach_Controller-rescue:GND-power #PWR0130
 U 1 1 5F19E154
 P 5850 4450
@@
 $EndComp
 $Comp
-L power:GND #PWR0132
+L Gouach_Controller-rescue:GND-power #PWR0132
 U 1 1 5F19EFD3
 P 7200 4250
@@
 $EndComp
 $Comp
-L Device:C C4
+L Gouach_Controller-rescue:C-Device C4
 U 1 1 53F59FA3
 P 7200 4100
@@
 F 0 "C4" H 7200 4200 50  0000 L CNN
 F 1 "100nF" H 7206 4015 50  0000 L CNN
-F 2 "Capacitors_SMD:C_0603" H 7238 3950 30  0001 C CNN
+F 2 "Capacitor_SMD:C_0603_1608Metric" H 7238 3950 30  0001 C CNN
 F 3 "" H 7200 4100 60  0000 C CNN
 F 4 "50V" H 7200 4100 50  0001 C CNN "Tension"

Commit message: Add Mouser order number
Parts:
- U4: Mouser (none) -> 595-SN65HVD232DR; mfg# SN65HVD232 -> (none)
Changed lines of the file:
@@
 F 1 "SN65HVD232" H 5900 3700 50  0000 C CNN
 F 2 "Package_SO:SOIC-8_3.9x4.9mm_P1.27mm" H 5850 4050 35  0001 C CIN
-F 3 "SN65HVD232" H 5850 4050 60  0001 C CNN
-F 4 "SN65HVD232" H 5850 4050 50  0001 C CNN "mfg#"
+F 3 "http://www.ti.com/lit/ds/symlink/sn65hvd230.pdf" H 5850 4050 60  0001 C CNN
+F 4 "" H 5850 4050 50  0001 C CNN "mfg#"
+F 5 "595-SN65HVD232DR" H 5850 4050 50  0001 C CNN "Mouser"
 	1    5850 4050
 	-1   0    0    -1
