File: Kicad/Gouach_Controller.kicad_pcb (KiCad board)
At the start: 4 copper layers, 41 x 104 mm, 139 parts, among them J1 HALL/Encoder, J10 USB, J11 CAN, J12 Serial, J2 Peripherals, J3 Peripherals, J4 BAT+, J5 BAT-, J6 M1, J7 M2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

Commit message: Add Mouser order number
Parts:
- C22, C24: value NP -> (none)
- G***: value LOGO -> (none)
Changed lines of the file:
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@@
     (descr "Capacitor SMD 0603 (1608 Metric), square (rectangular) end terminal, IPC_7351 nominal, (Body size source: http://www.tortai-tech.com/upload/download/2011102023233369053.pdf), generated with kicad-footprint-generator")
     (tags capacitor)
-    (attr smd)
+    (attr virtual)
     (fp_text reference C24 (at 0 -1.2065) (layer F.SilkS)
       (effects (font (size 0.7 0.7) (thickness 0.1)))
     )
-    (fp_text value NP (at 0 1.43) (layer F.Fab)
+    (fp_text value " " (at 0 1.43) (layer F.Fab)
       (effects (font (size 0.7 0.7) (thickness 0.1)))
     )
@@
     (descr "Capacitor SMD 0603 (1608 Metric), square (rectangular) end terminal, IPC_7351 nominal, (Body size source: http://www.tortai-tech.com/upload/download/2011102023233369053.pdf), generated with kicad-footprint-generator")
     (tags capacitor)
-    (attr smd)
+    (attr virtual)
     (fp_text reference C22 (at 0 -1.27) (layer F.SilkS)
       (effects (font (size 0.7 0.7) (thickness 0.1)))
     )
-    (fp_text value NP (at 0 1.43) (layer F.Fab)
+    (fp_text value " " (at 0 1.43) (layer F.Fab)
       (effects (font (size 0.7 0.7) (thickness 0.1)))
     )
@@
     (descr "Through hole straight pin header, 1x02, 2.54mm pitch, single row")
     (tags "Through hole pin header THT 1x02 2.54mm single row")
+    (attr virtual)
     (fp_text reference J11 (at 2.2225 1.0795 180) (layer F.SilkS) hide
       (effects (font (size 0.7 0.7) (thickness 0.1)))
@@
     (descr "Through hole straight pin header, 1x04, 2.54mm pitch, single row")
     (tags "Through hole pin header THT 1x04 2.54mm single row")
+    (attr virtual)
     (fp_text reference J10 (at 1.905 3.7465 180) (layer F.SilkS) hide
       (effects (font (size 0.7 0.7) (thickness 0.1)))
@@
     (descr "Through hole straight pin header, 2x03, 2.54mm pitch, double rows")
     (tags "Through hole pin header THT 2x03 2.54mm double row")
+    (attr virtual)
     (fp_text reference J1 (at 1.27 3.81) (layer F.SilkS) hide
       (effects (font (size 0.7 0.7) (thickness 0.1)))
@@
       (effects (font (size 0.7 0.7) (thickness 0.1)) (justify mirror))
     )
-    (fp_text value LOGO (at 0.75 0) (layer B.SilkS) hide
+    (fp_text value "" (at 0.75 0) (layer B.SilkS) hide
       (effects (font (size 0.7 0.7) (thickness 0.1)) (justify mirror))
     )
