File: Kicad/Gouach_Controller.kicad_pcb (KiCad board)
At the start: 4 copper layers, 41 x 104 mm, 139 parts, among them J1 HALL/Encoder, J10 USB, J11 CAN, J12 Serial, J2 Peripherals, J3 Peripherals, J4 BAT+, J5 BAT-, J6 M1, J7 M2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

Commit message: Add HTML BOM
Parts:
- C48: value 15uF -> EEUFS1K391B
- R22: value 2k2 -> 100R
Changed lines of the file:
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@@
       (usegerberadvancedattributes false)
       (creategerberjobfile false)
-      (excludeedgelayer true)
+      (excludeedgelayer false)
       (linewidth 0.150000)
       (plotframeref false)
@@
   (module Gouach-Controller:Capacitor_Horizontal (layer F.Cu)
     (at 109.525 52.083 270)
-    (attr virtual)
     (fp_text reference C48 (at 0 0 270) (layer F.SilkS) hide
       (effects (font (size 0.7 0.7) (thickness 0.1)))
     )
-    (fp_text value 15uF (at 0 -1.9 270) (layer F.Fab)
+    (fp_text value EEUFS1K391B (at 0 -1.9 270) (layer F.Fab)
       (effects (font (size 0.7 0.7) (thickness 0.1)))
     )
@@
       (effects (font (size 0.7 0.7) (thickness 0.1)))
     )
-    (fp_text value 2k2 (at 0 1.43) (layer F.Fab)
-      (effects (font (size 0.7 0.7) (thickness 0.1)))
-    )
+    (fp_text value 100R (at 0 1.43) (layer F.Fab)
+      (effects (font (size 0.7 0.7) (thickness 0.1)))
+    )
