File: Kicad/GC - Power.sch (KiCad schematic (older format))
At the start: 18 parts, among them U2 TC2117, U5 TPS54360DDA

Commit message: Passives changed from 0805 to 0603
Parts:
- removed C47: 15uF/100V, Capacitors_Tantalum_SMD:CP_Tantalum_Case-B_EIA-3528-21_Reflow, symbol Device:CP1
- removed U2: TC2117, TO_SOT_Packages_SMD:SOT-223-3_TabPin2, symbol regul:NCP1117-3.3_SOT223
- added C47: 10uF, Capacitors_SMD:C_0603, symbol Device:C
- added U2: XC6220B331MR, TO_SOT_Packages_SMD:SOT-23-5, symbol Regulator_Linear:XC6220B331MR
- C46: value 2.2uF -> 10uF; footprint Capacitors_SMD:C_0805 -> Capacitors_SMD:C_0603
- C51, C52, C53: footprint Capacitors_SMD:C_0805 -> Capacitors_SMD:C_0603
- R17, R44, R45, R5: footprint Resistors_SMD:R_0805 -> Resistors_SMD:R_0603
Connections:
- wire segments 63 -> 64
- no-connect marks 0 -> 1
Other:
- moved on the sheet: C46
Changed lines of the file:
@@
 L Device:C C?
 U 1 1 50500B3A
-P 6300 4900
+P 6900 3950
 AR Path="/50500B3A" Ref="C?"  Part="1"
 AR Path="/5E3AB6B4/50500B3A" Ref="C46"  Part="1"
-F 0 "C46" H 6415 4946 50  0000 L CNN
-F 1 "2.2uF" H 6415 4855 50  0000 L CNN
-F 2 "Capacitors_SMD:C_0805" H 6300 4900 60  0001 C CNN
-F 3 "" H 6300 4900 60  0001 C CNN
-	1    6300 4900
-	1    0    0    -1
-$EndComp
-$Comp
-L Device:CP1 C47
-U 1 1 50500B52
-P 6800 4900
-F 0 "C47" H 6915 4946 50  0000 L CNN
-F 1 "15uF/100V" H 6915 4855 50  0000 L CNN
-F 2 "Capacitors_Tantalum_SMD:CP_Tantalum_Case-B_EIA-3528-21_Reflow" H 6800 4900 60  0001 C CNN
-F 3 "" H 6800 4900 60  0001 C CNN
-	1    6800 4900
-	1    0    0    -1
-$EndComp
-$Comp
-L regul:NCP1117-3.3_SOT223 U2
-U 1 1 53E7AF36
-P 5900 4700
-F 0 "U2" H 5900 4942 50  0000 C CNN
-F 1 "TC2117" H 5900 4851 50  0000 C CNN
-F 2 "TO_SOT_Packages_SMD:SOT-223-3_TabPin2" H 5900 4700 60  0001 C CNN
-F 3 "NCP1117-3.3" H 5900 4700 60  0001 C CNN
-F 4 "NCP1117-3.3" H 5900 4700 50  0001 C CNN "mfg#"
-	1    5900 4700
-	1    0    0    -1
-$EndComp
-Wire Wire Line
-	6300 4700 6300 4750
-Connection ~ 6300 5100
-Wire Wire Line
-	6800 5100 6800 5050
-Wire Wire Line
-	6300 5100 6300 5050
-Connection ~ 5900 5100
-Wire Wire Line
-	6800 4700 6800 4650
-Wire Wire Line
-	6800 4700 6800 4750
-Connection ~ 6800 4700
-Wire Wire Line
-	5600 4700 5500 4700
-Wire Wire Line
-	5500 4700 5500 4650
-Wire Wire Line
-	6300 5100 6800 5100
-Wire Wire Line
-	5900 5100 6300 5100
-Wire Wire Line
-	5900 5100 5900 5150
-Wire Wire Line
-	6300 4700 6800 4700
+F 0 "C46" H 7015 3996 50  0000 L CNN
+F 1 "10uF" H 7015 3905 50  0000 L CNN
+F 2 "Capacitors_SMD:C_0603" H 6900 3950 60  0001 C CNN
+F 3 "" H 6900 3950 60  0001 C CNN
+	1    6900 3950
+	1    0    0    -1
+$EndComp
 $Comp
 L power:+3V3 #PWR0171
 U 1 1 5F178995
-P 6800 4650
-F 0 "#PWR0171" H 6800 4500 50  0001 C CNN
-F 1 "+3V3" H 6800 4800 50  0000 C CNN
-F 2 "" H 6800 4650 50  0001 C CNN
-F 3 "" H 6800 4650 50  0001 C CNN
-	1    6800 4650
+P 6900 3650
+F 0 "#PWR0171" H 6900 3500 50  0001 C CNN
+F 1 "+3V3" H 6900 3800 50  0000 C CNN
+F 2 "" H 6900 3650 50  0001 C CNN
+F 3 "" H 6900 3650 50  0001 C CNN
+	1    6900 3650
 	1    0    0    -1
 $EndComp
@@
 L power:+5V #PWR0172
 U 1 1 5F179269
-P 5500 4650
-F 0 "#PWR0172" H 5500 4500 50  0001 C CNN
-F 1 "+5V" H 5500 4800 50  0000 C CNN
-F 2 "" H 5500 4650 50  0001 C CNN
-F 3 "" H 5500 4650 50  0001 C CNN
-	1    5500 4650
+P 5650 3650
+F 0 "#PWR0172" H 5650 3500 50  0001 C CNN
+F 1 "+5V" H 5650 3800 50  0000 C CNN
+F 2 "" H 5650 3650 50  0001 C CNN
+F 3 "" H 5650 3650 50  0001 C CNN
+	1    5650 3650
 	1    0    0    -1
 $EndComp
@@
 L power:GND #PWR0173
 U 1 1 5F17A322
-P 5900 5150
-F 0 "#PWR0173" H 5900 4900 50  0001 C CNN
-F 1 "GND" H 5900 5000 50  0000 C CNN
-F 2 "" H 5900 5150 50  0001 C CNN
-F 3 "" H 5900 5150 50  0001 C CNN
-	1    5900 5150
+P 6350 4250
+F 0 "#PWR0173" H 6350 4000 50  0001 C CNN
+F 1 "GND" H 6350 4100 50  0000 C CNN
+F 2 "" H 6350 4250 50  0001 C CNN
+F 3 "" H 6350 4250 50  0001 C CNN
+	1    6350 4250
 	1    0    0    -1
 $EndComp
@@
 	-1   0    0    1
 $EndComp
-Wire Wire Line
-	6200 4700 6300 4700
-Connection ~ 6300 4700
 $Comp
 L power:PWR_FLAG #FLG0103
 U 1 1 5F17F61E
+P 1850 7050
+F 0 "#FLG0103" H 1850 7125 50  0001 C CNN
+F 1 "PWR_FLAG" V 1850 7350 50  0000 C CNN
+F 2 "" H 1850 7050 50  0001 C CNN
+F 3 "~" H 1850 7050 50  0001 C CNN
+	1    1850 7050
+	-1   0    0    1
+$EndComp
+$Comp
+L power:GND #PWR0174
+U 1 1 5F17B34C
+P 1850 7050
+F 0 "#PWR0174" H 1850 6800 50  0001 C CNN
+F 1 "GND" H 1850 6900 50  0000 C CNN
+F 2 "" H 1850 7050 50  0001 C CNN
+F 3 "" H 1850 7050 50  0001 C CNN
+	1    1850 7050
+	-1   0    0    1
+$EndComp
+$Comp
+L power:+3V3 #PWR0110
+U 1 1 5F59F4EE
 P 1600 7050
-F 0 "#FLG0103" H 1600 7125 50  0001 C CNN
+F 0 "#PWR0110" H 1600 6900 50  0001 C CNN
+F 1 "+3V3" H 1600 7200 50  0000 C CNN
+F 2 "" H 1600 7050 50  0001 C CNN
+F 3 "" H 1600 7050 50  0001 C CNN
+	1    1600 7050
+	1    0    0    -1
+$EndComp
+$Comp
+L power:PWR_FLAG #FLG0102
+U 1 1 5F5A0DF0
+P 1600 7050
+F 0 "#FLG0102" H 1600 7125 50  0001 C CNN
 F 1 "PWR_FLAG" V 1600 7350 50  0000 C CNN
 F 2 "" H 1600 7050 50  0001 C CNN
 F 3 "~" H 1600 7050 50  0001 C CNN
 	1    1600 7050
-	-1   0    0    1
-$EndComp
-$Comp
-L power:GND #PWR0174
-U 1 1 5F17B34C
-P 1600 7050
-F 0 "#PWR0174" H 1600 6800 50  0001 C CNN
-F 1 "GND" H 1600 6900 50  0000 C CNN
-F 2 "" H 1600 7050 50  0001 C CNN
-F 3 "" H 1600 7050 50  0001 C CNN
-	1    1600 7050
-	-1   0    0    1
-$EndComp
-Wire Wire Line
-	5900 5000 5900 5100
-$Comp
-L power:+3V3 #PWR0110
-U 1 1 5F59F4EE
-P 1350 7050
-F 0 "#PWR0110" H 1350 6900 50  0001 C CNN
-F 1 "+3V3" H 1350 7200 50  0000 C CNN
-F 2 "" H 1350 7050 50  0001 C CNN
-F 3 "" H 1350 7050 50  0001 C CNN
-	1    1350 7050
-	1    0    0    -1
-$EndComp
-$Comp
-L power:PWR_FLAG #FLG0102
-U 1 1 5F5A0DF0
-P 1350 7050
-F 0 "#FLG0102" H 1350 7125 50  0001 C CNN
-F 1 "PWR_FLAG" V 1350 7350 50  0000 C CNN
-F 2 "" H 1350 7050 50  0001 C CNN
-F 3 "~" H 1350 7050 50  0001 C CNN
-	1    1350 7050
 	-1   0    0    1
 $EndComp
@@
 F 0 "C52" H 7250 2350 50  0000 L CNN
 F 1 "51pF" H 7200 2250 50  0000 L CNN
-F 2 "Capacitors_SMD:C_0805" H 7500 2300 60  0001 C CNN
+F 2 "Capacitors_SMD:C_0603" H 7500 2300 60  0001 C CNN
 F 3 "" H 7500 2300 60  0001 C CNN
 	1    7500 2300
@@
 F 0 "C53" H 7915 2496 50  0000 L CNN
 F 1 "1.8nF" H 7915 2405 50  0000 L CNN
-F 2 "Capacitors_SMD:C_0805" H 7800 2450 60  0001 C CNN
+F 2 "Capacitors_SMD:C_0603" H 7800 2450 60  0001 C CNN
 F 3 "" H 7800 2450 60  0001 C CNN
 	1    7800 2450
@@
 AR Path="/5E3F36E9" Ref="C?"  Part="1"
 AR Path="/5E3AB6B4/5E3F36E9" Ref="C51"  Part="1"
-F 0 "C51" H 6700 1850 50  0000 L CNN
-F 1 "100nF" H 6700 1650 50  0000 L CNN
-F 2 "Capacitors_SMD:C_0805" H 6650 1750 60  0001 C CNN
+F 0 "C51" H 6700 1950 50  0000 L CNN
+F 1 "100nF" H 6700 1850 50  0000 L CNN
+F 2 "Capacitors_SMD:C_0603" H 6650 1750 60  0001 C CNN
 F 3 "" H 6650 1750 60  0001 C CNN
 	1    6650 1750
@@
 F 0 "R45" H 7730 2104 50  0000 R CNN
 F 1 "15.4k" H 7730 2195 50  0000 R CNN
-F 2 "Resistors_SMD:R_0805" V 7730 2150 50  0001 C CNN
+F 2 "Resistors_SMD:R_0603" V 7730 2150 50  0001 C CNN
 F 3 "" H 7800 2150 50  0001 C CNN
 	1    7800 2150
@@
 F 0 "R5" H 5520 2246 50  0000 L CNN
 F 1 "274k" H 5520 2155 50  0000 L CNN
-F 2 "Resistors_SMD:R_0805" V 5380 2200 50  0001 C CNN
+F 2 "Resistors_SMD:R_0603" V 5380 2200 50  0001 C CNN
 F 3 "" H 5450 2200 50  0001 C CNN
 	1    5450 2200
@@
 F 0 "R17" H 7220 2146 50  0000 L CNN
 F 1 "60.4k" H 7220 2055 50  0000 L CNN
-F 2 "Resistors_SMD:R_0805" V 7080 2100 50  0001 C CNN
+F 2 "Resistors_SMD:R_0603" V 7080 2100 50  0001 C CNN
 F 3 "" H 7150 2100 50  0001 C CNN
 	1    7150 2100
@@
 F 0 "R44" H 7220 2496 50  0000 L CNN
 F 1 "11.5k" H 7220 2405 50  0000 L CNN
-F 2 "Resistors_SMD:R_0805" V 7080 2450 50  0001 C CNN
+F 2 "Resistors_SMD:R_0603" V 7080 2450 50  0001 C CNN
 F 3 "" H 7150 2450 50  0001 C CNN
 	1    7150 2450
@@
 U 1 1 5E3F69F6
 P 6900 1900
-F 0 "L2" V 7090 1900 50  0000 C CNN
-F 1 "10uH" V 6999 1900 50  0000 C CNN
+F 0 "L2" V 7000 1900 50  0000 C CNN
+F 1 "10uH" V 6850 1900 50  0000 C CNN
 F 2 "Inductors_SMD:L_Coilcraft_XAL5030" H 6900 1900 50  0001 C CNN
 F 3 "XAL5050-103MEB" H 6900 1900 50  0001 C CNN
@@
 Wire Wire Line
 	6250 2650 6150 2650
+NoConn ~ 5750 2200
+$Comp
+L power:+5VP #PWR0106
+U 1 1 5E51FB26
+P 1350 7050
+F 0 "#PWR0106" H 1350 6900 50  0001 C CNN
+F 1 "+5VP" H 1350 7200 50  0000 C CNN
+F 2 "" H 1350 7050 50  0001 C CNN
+F 3 "" H 1350 7050 50  0001 C CNN
+	1    1350 7050
+	1    0    0    -1
+$EndComp
+$Comp
+L power:PWR_FLAG #FLG0105
+U 1 1 5E5211E0
+P 1350 7050
+F 0 "#FLG0105" H 1350 7125 50  0001 C CNN
+F 1 "PWR_FLAG" V 1350 7350 50  0000 C CNN
+F 2 "" H 1350 7050 50  0001 C CNN
+F 3 "~" H 1350 7050 50  0001 C CNN
+	1    1350 7050
+	-1   0    0    1
+$EndComp
+$Comp
+L Regulator_Linear:XC6220B331MR U2
+U 1 1 5E533A67
+P 6350 3800
+F 0 "U2" H 6350 4167 50  0000 C CNN
+F 1 "XC6220B331MR" H 6350 4076 50  0000 C CNN
+F 2 "TO_SOT_Packages_SMD:SOT-23-5" H 6350 3800 50  0001 C CNN
+F 3 "https://www.torexsemi.com/file/xc6220/XC6220.pdf" H 7100 2800 50  0001 C CNN
+	1    6350 3800
+	1    0    0    -1
+$EndComp
+$Comp
+L Device:C C?
+U 1 1 5E535C87
+P 5650 3950
+AR Path="/5E535C87" Ref="C?"  Part="1"
+AR Path="/5E3AB6B4/5E535C87" Ref="C47"  Part="1"
+F 0 "C47" H 5765 3996 50  0000 L CNN
+F 1 "10uF" H 5765 3905 50  0000 L CNN
+F 2 "Capacitors_SMD:C_0603" H 5650 3950 60  0001 C CNN
+F 3 "" H 5650 3950 60  0001 C CNN
+	1    5650 3950
+	-1   0    0    -1
+$EndComp
+Wire Wire Line
+	5850 3900 5800 3900
+Wire Wire Line
+	5800 3900 5800 3700
+Wire Wire Line
+	5800 3700 5850 3700
+Connection ~ 5800 3700
+Wire Wire Line
+	5650 3650 5650 3700
+Wire Wire Line
+	5650 4100 5650 4200
+Wire Wire Line
+	5650 4200 6350 4200
+Wire Wire Line
+	6350 4200 6900 4200
+Wire Wire Line
+	6900 4200 6900 4100
+Connection ~ 6350 4200
+Wire Wire Line
+	5650 3800 5650 3700
+Connection ~ 5650 3700
+Wire Wire Line
+	5650 3700 5800 3700
+Wire Wire Line
+	6850 3700 6900 3700
+Wire Wire Line
+	6900 3700 6900 3800
+Wire Wire Line
+	6900 3700 6900 3650
+Connection ~ 6900 3700
+Wire Wire Line
+	6350 4200 6350 4250
 $EndSCHEMATC

Commit message: Components placed
Parts:
- C3, C49, C50: footprint Capacitors_SMD:C_2220 -> Capacitors_SMD:C_1210
- D6: value 100V -> 60V; footprint TO_SOT_Packages_SMD:TO-277A -> Diodes_SMD:D_SOD-123F; mfg# (none) -> PMEG6020ER-115
Changed lines of the file:
@@
 F 0 "C50" H 5000 2250 50  0000 L CNN
 F 1 "10uF" H 4950 2050 50  0000 L CNN
-F 2 "Capacitors_SMD:C_2220" H 5150 2150 60  0001 C CNN
+F 2 "Capacitors_SMD:C_1210" H 5150 2150 60  0001 C CNN
 F 3 "" H 5150 2150 60  0001 C CNN
 	1    5150 2150
@@
 F 0 "C49" H 4700 2250 50  0000 L CNN
 F 1 "10uF" H 4650 2050 50  0000 L CNN
-F 2 "Capacitors_SMD:C_2220" H 4850 2150 60  0001 C CNN
+F 2 "Capacitors_SMD:C_1210" H 4850 2150 60  0001 C CNN
 F 3 "" H 4850 2150 60  0001 C CNN
 	1    4850 2150
@@
 F 0 "C3" H 4450 2250 50  0000 L CNN
 F 1 "10uF" H 4350 2050 50  0000 L CNN
-F 2 "Capacitors_SMD:C_2220" H 4550 2150 60  0001 C CNN
+F 2 "Capacitors_SMD:C_1210" H 4550 2150 60  0001 C CNN
 F 3 "" H 4550 2150 60  0001 C CNN
 	1    4550 2150
@@
 P 6700 2100
 F 0 "D6" V 6654 2179 50  0000 L CNN
-F 1 "100V" V 6745 2179 50  0000 L CNN
-F 2 "TO_SOT_Packages_SMD:TO-277A" H 6700 2100 50  0001 C CNN
-F 3 "~" H 6700 2100 50  0001 C CNN
+F 1 "60V" V 6745 2179 50  0000 L CNN
+F 2 "Diodes_SMD:D_SOD-123F" H 6700 2100 50  0001 C CNN
+F 3 "PMEG6020ER-115" H 6700 2100 50  0001 C CNN
+F 4 "PMEG6020ER-115" H 6700 2100 50  0001 C CNN "mfg#"
 	1    6700 2100
 	0    1    1    0

Commit message: Adjusting capacitor size/value
Parts:
- C3, C49, C50: footprint Capacitors_SMD:C_1210 -> Capacitors_SMD:C_1206; Tension (none) -> 100V
- C46, C47: Tension (none) -> 25V
- C48: value 15uF/100V -> 15uF; footprint Capacitors_THT:CP_Radial_D8.0mm_P3.80mm -> Romain:Capacitor_Horizontal; Tension (none) -> 100V
- C51, C52, C53: Tension (none) -> 50V
- C54: Tension (none) -> 10V
Connections:
- net labels added: VBUS
- net labels removed: +5VP
Changed lines of the file:
@@
 F 2 "Capacitors_SMD:C_0603" H 6900 3950 60  0001 C CNN
 F 3 "" H 6900 3950 60  0001 C CNN
+F 4 "25V" H 6900 3950 50  0001 C CNN "Tension"
 	1    6900 3950
 	1    0    0    -1
@@
 P 3550 4950
 F 0 "C48" H 3665 4996 50  0000 L CNN
-F 1 "15uF/100V" H 3665 4905 50  0000 L CNN
-F 2 "Capacitors_THT:CP_Radial_D8.0mm_P3.80mm" H 3550 4950 60  0001 C CNN
+F 1 "15uF" H 3665 4905 50  0000 L CNN
+F 2 "Romain:Capacitor_Horizontal" H 3550 4950 60  0001 C CNN
 F 3 "" H 3550 4950 60  0001 C CNN
+F 4 "100V" H 3550 4950 50  0001 C CNN "Tension"
 	1    3550 4950
 	1    0    0    -1
@@
 F 0 "C50" H 5000 2250 50  0000 L CNN
 F 1 "10uF" H 4950 2050 50  0000 L CNN
-F 2 "Capacitors_SMD:C_1210" H 5150 2150 60  0001 C CNN
+F 2 "Capacitors_SMD:C_1206" H 5150 2150 60  0001 C CNN
 F 3 "" H 5150 2150 60  0001 C CNN
+F 4 "100V" H 5150 2150 50  0001 C CNN "Tension"
 	1    5150 2150
 	1    0    0    -1
@@
 F 0 "C49" H 4700 2250 50  0000 L CNN
 F 1 "10uF" H 4650 2050 50  0000 L CNN
-F 2 "Capacitors_SMD:C_1210" H 4850 2150 60  0001 C CNN
+F 2 "Capacitors_SMD:C_1206" H 4850 2150 60  0001 C CNN
 F 3 "" H 4850 2150 60  0001 C CNN
+F 4 "100V" H 4850 2150 50  0001 C CNN "Tension"
 	1    4850 2150
 	1    0    0    -1
@@
 F 0 "C3" H 4450 2250 50  0000 L CNN
 F 1 "10uF" H 4350 2050 50  0000 L CNN
-F 2 "Capacitors_SMD:C_1210" H 4550 2150 60  0001 C CNN
+F 2 "Capacitors_SMD:C_1206" H 4550 2150 60  0001 C CNN
 F 3 "" H 4550 2150 60  0001 C CNN
+F 4 "100V" H 4550 2150 50  0001 C CNN "Tension"
 	1    4550 2150
 	1    0    0    -1
@@
 F 2 "Capacitors_SMD:C_0603" H 7500 2300 60  0001 C CNN
 F 3 "" H 7500 2300 60  0001 C CNN
+F 4 "50V" H 7500 2300 50  0001 C CNN "Tension"
 	1    7500 2300
 	-1   0    0    -1
@@
 F 2 "Capacitors_SMD:C_0603" H 7800 2450 60  0001 C CNN
 F 3 "" H 7800 2450 60  0001 C CNN
+F 4 "50V" H 7800 2450 50  0001 C CNN "Tension"
 	1    7800 2450
 	1    0    0    -1
@@
 F 2 "Capacitors_SMD:C_0603" H 6650 1750 60  0001 C CNN
 F 3 "" H 6650 1750 60  0001 C CNN
+F 4 "50V" H 6650 1750 50  0001 C CNN "Tension"
 	1    6650 1750
 	1    0    0    -1
@@
 F 2 "Capacitors_SMD:CP_Elec_5x5.8" H 8100 2250 60  0001 C CNN
 F 3 "" H 8100 2250 60  0001 C CNN
+F 4 "10V" H 8100 2250 50  0001 C CNN "Tension"
 	1    8100 2250
 	1    0    0    -1
@@
 	6600 2300 7150 2300
 $Comp
-L power:+5VP #PWR09
+L power:VBUS #PWR09
 U 1 1 5E434096
 P 8100 1850
 F 0 "#PWR09" H 8100 1700 50  0001 C CNN
-F 1 "+5VP" H 8100 2000 50  0000 C CNN
+F 1 "VBUS" H 8100 2000 50  0000 C CNN
 F 2 "" H 8100 1850 50  0001 C CNN
 F 3 "" H 8100 1850 50  0001 C CNN
@@
 NoConn ~ 5750 2200
 $Comp
-L power:+5VP #PWR0106
+L power:VBUS #PWR0106
 U 1 1 5E51FB26
 P 1350 7050
 F 0 "#PWR0106" H 1350 6900 50  0001 C CNN
-F 1 "+5VP" H 1350 7200 50  0000 C CNN
+F 1 "VBUS" H 1350 7200 50  0000 C CNN
 F 2 "" H 1350 7050 50  0001 C CNN
 F 3 "" H 1350 7050 50  0001 C CNN
@@
 F 2 "Capacitors_SMD:C_0603" H 5650 3950 60  0001 C CNN
 F 3 "" H 5650 3950 60  0001 C CNN
+F 4 "25V" H 5650 3950 50  0001 C CNN "Tension"
 	1    5650 3950
 	-1   0    0    -1
