File: Kicad/Gouach_Controller.sch (KiCad schematic (older format))
At the start: 24 parts, among them J1 HALL/Encoder, J10 USB, J11 CANBUS, J12 Serial, J3 Peripherals, J4 IN+, J5 IN-, J6 MOTOR3, J7 MOTOR2, J8 MOTOR1

Commit message: Passives changed from 0805 to 0603
Parts:
- added J2: Peripherals, Romain:TerminalBlock_Phoenix_MPT-2.54mm_7pol, symbol conn:Conn_01x07
- C2: footprint Capacitors_SMD:C_0805 -> Capacitors_SMD:C_0603
- D1, D2, D3: footprint LEDs:LED_0805 -> LEDs:LED_0603
- J11: footprint Pin_Headers:Pin_Header_Straight_1x04_Pitch2.54mm -> Pin_Headers:Pin_Header_Straight_1x02_Pitch2.54mm; symbol conn:Conn_01x04 -> conn:Conn_01x02
- J3: footprint Romain:TBL009-254-16BE-2BE -> Romain:TerminalBlock_Phoenix_MPT-2.54mm_7pol; symbol conn:Conn_01x16 -> conn:Conn_01x07
- R103, R104, R22, R3, R37, R38, R4: footprint Resistors_SMD:R_0805 -> Resistors_SMD:R_0603
Other:
- moved on the sheet: C2, J12, R103, R104, R3, R4

Commit message: Components placed
Parts:
- removed R103, R104: 22R, Resistors_SMD:R_0603, symbol Device:R
- added Q7: DMN3300U, TO_SOT_Packages_SMD:SOT-23, symbol Transistor_FET:DMN3300U
- added R46: 100R, Resistors_SMD:R_0603, symbol Device:R
- added R47: 10k, Resistors_SMD:R_0603, symbol Device:R
- added U6: USBLC6-2SC6, TO_SOT_Packages_SMD:SOT-23-6, symbol Power_Protection:USBLC6-2SC6
Connections:
- net +5VP: now also Q7.3 (D), U6.5 (VBUS)
- net D+: now also J10.3 (Pin_3), U6.3 (IO2); no longer J10.2 (Pin_2)
- net D-: now also J10.2 (Pin_2), U6.1 (IO1); no longer J10.3 (Pin_3)
- net GND: now also R47.2, U6.2 (GND)
- net MCU/USB_D+: now also U6.4 (IO2)
- net MCU/USB_D-: now also U6.6 (IO1)
- net at J3.6 (Pin_6): now also Q7.2 (S)
- new net: Q7.1 (G), R46.2, R47.1
- new net MCU/LAMP_CMD: R46.1
Other:
- moved on the sheet: C2, J1, J10, J11, J12, J2, J3, J6, J7, J8, R3, R4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

Commit message: Adjusted cap size/value + add ESD protection on USB
Parts:
- C2: Tension (none) -> 50V
- J11: value CANBUS -> CAN
- J4, J5: footprint Connectors:1pin -> Mounting_Holes:MountingHole_2.7mm_Pad_Via
- J6, J7, J8: footprint Connectors:1pin -> Mounting_Holes:MountingHole_2.2mm_M2_Pad_Via
Connections:
- net labels added: VBUS
- net labels removed: +5VP
- wire segments 111 -> 114
Other:
- note removed: "Connect signal ground and\npower ground in one place only"
- moved on the sheet: J1
Changed lines of the file:
@@
 F 0 "J5" H 9130 1450 50  0000 L CNN
 F 1 "IN-" H 9050 1505 30  0001 C CNN
-F 2 "Connectors:1pin" H 9050 1450 60  0001 C CNN
+F 2 "Mounting_Holes:MountingHole_2.7mm_Pad_Via" H 9050 1450 60  0001 C CNN
 F 3 "" H 9050 1450 60  0001 C CNN
 	1    9050 1450
@@
 F 0 "J4" H 9130 1300 50  0000 L CNN
 F 1 "IN+" H 9050 1355 30  0001 C CNN
-F 2 "Connectors:1pin" H 9050 1300 60  0001 C CNN
+F 2 "Mounting_Holes:MountingHole_2.7mm_Pad_Via" H 9050 1300 60  0001 C CNN
 F 3 "" H 9050 1300 60  0001 C CNN
 	1    9050 1300
@@
 F 0 "J6" H 10300 2850 50  0000 L CNN
 F 1 "MOTOR3" H 10250 2905 30  0001 C CNN
-F 2 "Connectors:1pin" H 10250 2850 60  0001 C CNN
+F 2 "Mounting_Holes:MountingHole_2.2mm_M2_Pad_Via" H 10250 2850 60  0001 C CNN
 F 3 "" H 10250 2850 60  0001 C CNN
 	1    10250 2850
@@
 F 0 "J7" H 10300 3000 50  0000 L CNN
 F 1 "MOTOR2" H 10250 3055 30  0001 C CNN
-F 2 "Connectors:1pin" H 10250 3000 60  0001 C CNN
+F 2 "Mounting_Holes:MountingHole_2.2mm_M2_Pad_Via" H 10250 3000 60  0001 C CNN
 F 3 "" H 10250 3000 60  0001 C CNN
 	1    10250 3000
@@
 F 0 "J8" H 10300 3550 50  0000 L CNN
 F 1 "MOTOR1" H 10250 3605 30  0001 C CNN
-F 2 "Connectors:1pin" H 10250 3550 60  0001 C CNN
+F 2 "Mounting_Holes:MountingHole_2.2mm_M2_Pad_Via" H 10250 3550 60  0001 C CNN
 F 3 "" H 10250 3550 60  0001 C CNN
 	1    10250 3550
@@
 F26 "H2_VS" I R 7700 3500 60
 F27 "H3_VS" I R 7700 3600 60
-F28 "SH1_A" I R 7700 4250 60
-F29 "SH1_B" I R 7700 4450 60
-F30 "SH2_A" I R 7700 4750 60
-F31 "SH2_B" I R 7700 4950 60
+F28 "SH1+" I R 7700 4250 60
+F29 "SH1-" I R 7700 4450 60
+F30 "SH2+" I R 7700 4750 60
+F31 "SH2-" I R 7700 4950 60
 $EndSheet
 Connection ~ 7250 1900
@@
 Wire Wire Line
 	8200 3900 8200 4100
-Wire Wire Line
-	9550 4950 9550 5050
-Wire Wire Line
-	9850 4950 9850 5050
 Wire Wire Line
 	1550 2950 1950 2950
@@
 P 1350 2850
 F 0 "J11" H 1350 2950 50  0000 C CNN
-F 1 "CANBUS" V 1450 2800 50  0000 C CNN
+F 1 "CAN" V 1450 2800 50  0000 C CNN
 F 2 "Pin_Headers:Pin_Header_Straight_1x02_Pitch2.54mm" H 1350 2900 60  0001 C CNN
 F 3 "" H 1350 2900 60  0000 C CNN
@@
 	-1   0    0    -1
 $EndComp
-Wire Wire Line
-	9550 4950 9850 4950
 Wire Wire Line
 	2850 6400 3250 6400
@@
 F 4 "WSLP2726" H 8450 4850 50  0001 C CNN "mfg#"
 	1    8450 4850
-	-1   0    0    1
-$EndComp
-Text Notes 9150 4900 0    60   ~ 0
-Connect signal ground and\npower ground in one place only
+	-1   0    0    -1
+$EndComp
 Text Label 2200 4700 0    40   ~ 0
 ADC_TORQUE
@@
 L power:+5V #PWR0109
 U 1 1 5F1602A3
-P 1550 3400
-F 0 "#PWR0109" H 1550 3250 50  0001 C CNN
-F 1 "+5V" H 1550 3550 50  0000 C CNN
-F 2 "" H 1550 3400 50  0001 C CNN
-F 3 "" H 1550 3400 50  0001 C CNN
-	1    1550 3400
+P 1550 3350
+F 0 "#PWR0109" H 1550 3200 50  0001 C CNN
+F 1 "+5V" H 1550 3500 50  0000 C CNN
+F 2 "" H 1550 3350 50  0001 C CNN
+F 3 "" H 1550 3350 50  0001 C CNN
+	1    1550 3350
 	1    0    0    -1
 $EndComp
@@
 F 3 "" H 8450 5050 50  0001 C CNN
 	1    8450 5050
-	1    0    0    -1
-$EndComp
-$Comp
-L power:GND #PWR0116
-U 1 1 5F1966E1
-P 9550 5050
-F 0 "#PWR0116" H 9550 4800 50  0001 C CNN
-F 1 "GND" H 9550 4900 50  0000 C CNN
-F 2 "" H 9550 5050 50  0001 C CNN
-F 3 "" H 9550 5050 50  0001 C CNN
-	1    9550 5050
-	1    0    0    -1
-$EndComp
-$Comp
-L power:GND #PWR0117
-U 1 1 5F196A29
-P 9850 5050
-F 0 "#PWR0117" H 9850 4800 50  0001 C CNN
-F 1 "GND" H 9850 4900 50  0000 C CNN
-F 2 "" H 9850 5050 50  0001 C CNN
-F 3 "" H 9850 5050 50  0001 C CNN
-	1    9850 5050
 	1    0    0    -1
 $EndComp
@@
 L power:GND #PWR0124
 U 1 1 5F19975B
-P 1550 3800
-F 0 "#PWR0124" H 1550 3550 50  0001 C CNN
-F 1 "GND" V 1550 3600 50  0000 C CNN
-F 2 "" H 1550 3800 50  0001 C CNN
-F 3 "" H 1550 3800 50  0001 C CNN
-	1    1550 3800
+P 1550 3550
+F 0 "#PWR0124" H 1550 3300 50  0001 C CNN
+F 1 "GND" V 1550 3350 50  0000 C CNN
+F 2 "" H 1550 3550 50  0001 C CNN
+F 3 "" H 1550 3550 50  0001 C CNN
+	1    1550 3550
 	0    -1   -1   0
 $EndComp
@@
 L conn:Conn_01x06 J1
 U 1 1 522DA047
-P 1350 3600
-F 0 "J1" H 1350 3900 60  0000 C CNN
-F 1 "HALL/Encoder" V 1450 3550 60  0000 C CNN
-F 2 "Pin_Headers:Pin_Header_Straight_2x03_Pitch2.54mm" H 1350 3600 60  0001 C CNN
-F 3 "" H 1350 3600 60  0001 C CNN
-	1    1350 3600
+P 1350 3550
+F 0 "J1" H 1350 3850 60  0000 C CNN
+F 1 "HALL/Encoder" V 1450 3500 60  0000 C CNN
+F 2 "Pin_Headers:Pin_Header_Straight_2x03_Pitch2.54mm" H 1350 3550 60  0001 C CNN
+F 3 "" H 1350 3550 60  0001 C CNN
+	1    1350 3550
 	-1   0    0    -1
 $EndComp
@@
 F 2 "Capacitors_SMD:C_0603" H 6900 1900 60  0001 C CNN
 F 3 "" H 6900 1900 60  0001 C CNN
+F 4 "50V" H 6900 1900 50  0001 C CNN "Tension"
 	1    6900 1900
 	0    1    1    0
@@
 	1    0    0    -1
 $EndComp
-$Sheet
-S 1950 3350 850  600
-U 53FBA77E
-F0 "Filters" 50
-F1 "GC - Hall_Filters.sch" 50
-F2 "HALL3_IN" I L 1950 3800 40
-F3 "HALL2_IN" I L 1950 3700 40
-F4 "HALL1_IN" I L 1950 3500 40
-F5 "TEMP_IN" I L 1950 3600 40
-F6 "HALL3_OUT" O R 2800 3700 40
-F7 "HALL2_OUT" O R 2800 3600 40
-F8 "HALL1_OUT" O R 2800 3500 40
-F9 "TEMP_OUT" O R 2800 3800 40
-$EndSheet
 Text Label 1600 2000 0    50   ~ 0
 D+
@@
 $EndComp
 Wire Wire Line
-	1550 3500 1950 3500
-Wire Wire Line
-	1550 3600 1950 3600
-Wire Wire Line
-	1550 3700 1950 3700
-Wire Wire Line
-	1550 3900 1900 3900
-Wire Wire Line
-	1900 3900 1900 3800
+	1550 3850 1900 3850
+Wire Wire Line
+	1900 3850 1900 3800
 Wire Wire Line
 	1900 3800 1950 3800
 $Comp
-L power:+5VP #PWR0104
+L power:VBUS #PWR0104
 U 1 1 5E5514CA
 P 1550 1800
 F 0 "#PWR0104" H 1550 1650 50  0001 C CNN
-F 1 "+5VP" H 1550 1950 50  0000 C CNN
+F 1 "VBUS" H 1550 1950 50  0000 C CNN
 F 2 "" H 1550 1800 50  0001 C CNN
 F 3 "" H 1550 1800 50  0001 C CNN
@@
 	1750 5850 2400 5850
 $Comp
-L power:+5VP #PWR010
+L power:VBUS #PWR010
 U 1 1 5E51C46C
 P 2400 5450
 F 0 "#PWR010" H 2400 5300 50  0001 C CNN
-F 1 "+5VP" H 2400 5600 50  0000 C CNN
+F 1 "VBUS" H 2400 5600 50  0000 C CNN
 F 2 "" H 2400 5450 50  0001 C CNN
 F 3 "" H 2400 5450 50  0001 C CNN
@@
 $EndComp
 $Comp
-L power:+5VP #PWR0112
+L power:VBUS #PWR0112
 U 1 1 5E55D79F
 P 2900 1950
 F 0 "#PWR0112" H 2900 1800 50  0001 C CNN
-F 1 "+5VP" H 2900 2100 50  0000 C CNN
+F 1 "VBUS" H 2900 2100 50  0000 C CNN
 F 2 "" H 2900 1950 50  0001 C CNN
 F 3 "" H 2900 1950 50  0001 C CNN
@@
 F 4 "WSLP2726" H 7950 4350 50  0001 C CNN "mfg#"
 	1    7950 4350
-	-1   0    0    1
-$EndComp
+	-1   0    0    -1
+$EndComp
+$Sheet
+S 1950 3350 850  600
+U 53FBA77E
+F0 "Filters" 50
+F1 "GC - Hall_Filters.sch" 50
+F2 "HALL3_IN" I L 1950 3800 40
+F3 "HALL2_IN" I L 1950 3600 40
+F4 "HALL1_IN" I L 1950 3500 40
+F5 "TEMP_IN" I L 1950 3700 40
+F6 "HALL3_OUT" O R 2800 3700 40
+F7 "HALL2_OUT" O R 2800 3600 40
+F8 "HALL1_OUT" O R 2800 3500 40
+F9 "TEMP_OUT" O R 2800 3800 40
+$EndSheet
+Wire Wire Line
+	1550 3450 1800 3450
+Wire Wire Line
+	1800 3450 1800 3500
+Wire Wire Line
+	1800 3500 1950 3500
+Wire Wire Line
+	1550 3750 1850 3750
+Wire Wire Line
+	1850 3750 1850 3700
+Wire Wire Line
+	1850 3700 1950 3700
+Wire Wire Line
+	1550 3650 1800 3650
+Wire Wire Line
+	1800 3650 1800 3600
+Wire Wire Line
+	1800 3600 1950 3600
 $EndSCHEMATC

Commit message: Fixed libraries issues
Parts:
- C2: footprint Capacitors_SMD:C_0603 -> Capacitor_SMD:C_0603_1608Metric; symbol Device:C -> Gouach_Controller-rescue:C-Device
- D1, D2, D3: footprint LEDs:LED_0603 -> LED_SMD:LED_0603_1608Metric; symbol Device:LED -> Gouach_Controller-rescue:LED-Device
- H1: footprint Mounting_Holes:MountingHole_3.2mm_M3 -> MountingHole:MountingHole_3.2mm_M3; symbol Mechanical:MountingHole -> Gouach_Controller-rescue:MountingHole-Mechanical
- J1: footprint Pin_Headers:Pin_Header_Straight_2x03_Pitch2.54mm -> Connector_PinHeader_2.54mm:PinHeader_2x03_P2.54mm_Vertical; symbol conn:Conn_01x06 -> Gouach_Controller-rescue:Conn_01x06-conn
- J10, J12: footprint Pin_Headers:Pin_Header_Straight_1x04_Pitch2.54mm -> Connector_PinHeader_2.54mm:PinHeader_1x04_P2.54mm_Vertical; symbol conn:Conn_01x04 -> Gouach_Controller-rescue:Conn_01x04-conn
- J11: footprint Pin_Headers:Pin_Header_Straight_1x02_Pitch2.54mm -> Connector_PinHeader_2.54mm:PinHeader_1x02_P2.54mm_Vertical; symbol conn:Conn_01x02 -> Gouach_Controller-rescue:Conn_01x02-conn
- J2, J3: footprint Romain:TerminalBlock_Phoenix_MPT-2.54mm_7pol -> Gouach-Controller:TerminalBlock_Phoenix_MPT-2.54mm_7pol; symbol conn:Conn_01x07 -> Gouach_Controller-rescue:Conn_01x07-conn
- J4: value IN+ -> BAT+; footprint Mounting_Holes:MountingHole_2.7mm_Pad_Via -> MountingHole:MountingHole_2.7mm_Pad_Via; symbol conn:Conn_01x01 -> Gouach_Controller-rescue:Conn_01x01-conn
- J5: value IN- -> BAT-; footprint Mounting_Holes:MountingHole_2.7mm_Pad_Via -> MountingHole:MountingHole_2.7mm_Pad_Via; symbol conn:Conn_01x01 -> Gouach_Controller-rescue:Conn_01x01-conn
- J6: value MOTOR3 -> M1; footprint Mounting_Holes:MountingHole_2.2mm_M2_Pad_Via -> MountingHole:MountingHole_2.2mm_M2_Pad_Via; symbol conn:Conn_01x01 -> Gouach_Controller-rescue:Conn_01x01-conn
- J7: value MOTOR2 -> M2; footprint Mounting_Holes:MountingHole_2.2mm_M2_Pad_Via -> MountingHole:MountingHole_2.2mm_M2_Pad_Via; symbol conn:Conn_01x01 -> Gouach_Controller-rescue:Conn_01x01-conn
- J8: value MOTOR1 -> M3; footprint Mounting_Holes:MountingHole_2.2mm_M2_Pad_Via -> MountingHole:MountingHole_2.2mm_M2_Pad_Via; symbol conn:Conn_01x01 -> Gouach_Controller-rescue:Conn_01x01-conn
- Q7: footprint TO_SOT_Packages_SMD:SOT-23 -> Package_TO_SOT_SMD:SOT-23; symbol Transistor_FET:DMN3300U -> Gouach_Controller-rescue:DMN3300U-Transistor_FET
- R22, R3, R37, R38, R4, R46, R47: footprint Resistors_SMD:R_0603 -> Resistor_SMD:R_0603_1608Metric; symbol Device:R -> Gouach_Controller-rescue:R-Device
- R53, R54: footprint Romain:WSLP2726 -> Gouach-Controller:WSLP2726; symbol Device:R_Shunt -> Gouach_Controller-rescue:R_Shunt-Device
- U6: footprint TO_SOT_Packages_SMD:SOT-23-6 -> Package_TO_SOT_SMD:SOT-23-6; symbol Power_Protection:USBLC6-2SC6 -> Gouach_Controller-rescue:USBLC6-2SC6-Power_Protection

Commit message: Add Mouser order number
Parts:
- Q7: Mouser (none) -> 621-DMN3300U-7
- R53, R54: Mouser (none) -> 71-WSLP27261L000FEA; mfg# WSLP2726 -> (none)
- U6: Mouser (none) -> 511-USBLC6-2SC6
Changed lines of the file:
@@
 F 1 "1mR" V 8450 4850 50  0000 C CNN
 F 2 "Gouach-Controller:WSLP2726" H 8450 4850 60  0001 C CNN
-F 3 "WSLP2726" H 8450 4850 60  0001 C CNN
-F 4 "WSLP2726" H 8450 4850 50  0001 C CNN "mfg#"
+F 3 "https://www.vishay.com/docs/30179/wslp2726.pdf" H 8450 4850 60  0001 C CNN
+F 4 "" H 8450 4850 50  0001 C CNN "mfg#"
+F 5 "71-WSLP27261L000FEA " H 8450 4850 50  0001 C CNN "Mouser"
 	1    8450 4850
 	-1   0    0    -1
@@
 F 1 "MountingHole" H 1550 7105 50  0000 L CNN
 F 2 "MountingHole:MountingHole_3.2mm_M3" H 1450 7150 50  0001 C CNN
-F 3 "~" H 1450 7150 50  0001 C CNN
+F 3 "" H 1450 7150 50  0001 C CNN
 	1    1450 7150
 	1    0    0    -1
@@
 F 2 "Package_TO_SOT_SMD:SOT-23-6" H 1650 2350 50  0001 C CNN
 F 3 "http://www2.st.com/resource/en/datasheet/CD00050750.pdf" H 2600 2300 50  0001 C CNN
+F 4 "" H 2400 1950 50  0001 C CNN "mfg#"
+F 5 "511-USBLC6-2SC6" H 2400 1950 50  0001 C CNN "Mouser"
 	1    2400 1950
 	0    1    1    0
@@
 F 2 "Package_TO_SOT_SMD:SOT-23" H 2700 5575 50  0001 L CIN
 F 3 "http://www.diodes.com/assets/Datasheets/ds31181.pdf" H 2500 5650 50  0001 L CNN
+F 4 "" H 2500 5650 50  0001 C CNN "mfg#"
+F 5 "621-DMN3300U-7 " H 2500 5650 50  0001 C CNN "Mouser"
 	1    2500 5650
 	-1   0    0    -1
@@
 F 1 "1mR" V 7950 4350 50  0000 C CNN
 F 2 "Gouach-Controller:WSLP2726" H 7950 4350 60  0001 C CNN
-F 3 "WSLP2726" H 7950 4350 60  0001 C CNN
-F 4 "WSLP2726" H 7950 4350 50  0001 C CNN "mfg#"
+F 3 "https://www.vishay.com/docs/30179/wslp2726.pdf" H 7950 4350 60  0001 C CNN
+F 4 "" H 7950 4350 50  0001 C CNN "mfg#"
+F 5 "71-WSLP27261L000FEA " H 7950 4350 50  0001 C CNN "Mouser"
 	1    7950 4350
 	-1   0    0    -1

Commit message: Change R22 value
Parts:
- R22: value 2k2 -> 100R
Changed lines of the file:
@@
 P 6150 5500
 F 0 "R22" V 6050 5500 50  0000 C CNN
-F 1 "2k2" V 6150 5500 50  0000 C CNN
+F 1 "100R" V 6150 5500 50  0000 C CNN
 F 2 "Resistor_SMD:R_0603_1608Metric" H 6150 5500 60  0001 C CNN
 F 3 "" H 6150 5500 60  0001 C CNN
